File: RFM.sch (KiCad schematic (older format))
At the start: 43 parts

Commit message: Update
Parts:
- removed P?: USB_OTG, symbol USB_OTG
- removed P?: CONN_01X06, symbol CONN_01X06
- removed P? (x2): CONN_01X02, symbol CONN_01X02
- added J1: USB_OTG, symbol USB_OTG
- added J2: CONN_PWR, symbol CONN_01X02
- added J3: CONN_DEBUG, symbol CONN_01X06
- added J4: CONN_USART, symbol CONN_01X03
- added J5: CONN_SPI, symbol CONN_01X05
- C10, C11, C12, C13, C14, C15, C16, C17, C18, C19, C20, C21, C22, C23, C24, C7, C8, C9: renamed from C?; footprint (none) -> Capacitors_SMD:C_0402
- D1, D2: renamed from D?; footprint (none) -> LEDs:LED_0603
- R1, R2, R3, R4: renamed from R?; footprint (none) -> Resistors_SMD:R_0603
- U1: renamed from U?; value TPS79330 -> TPS79333
- Y1: renamed from Y?; footprint (none) -> Crystals:Crystal_SMD_0603-4pin_6.0x3.5mm
- Y2: renamed from Y?; footprint (none) -> Crystals:Crystal_AT310_d3.0mm_l10.0mm_Horizontal
- gave numbers to parts that had none: 12
Connections:
- net labels added: CC_GPIO0, CC_GPIO2, CC_GPIO3, CC_MISO, CC_MOSI, CC_NSS, CC_RESET_N, CC_SCLK, SPI_MISO, SPI_MOSI, SPI_NSS, SPI_SCK, USART_RX, USART_TX
- net labels removed: CSN, GPIO0, GPIO2, GPIO3, MISO, MOSI, RESET_N, SCLK, USART2_RX, USART2_TX
- wire segments 146 -> 157
- no-connect marks 1 -> 29
Other:
- note added: "Consider using LP38798"
- note added: "Linear regulator"
- note added: "TODO: Front end, GPS"
- note added: "TODO: decoupling"
- note removed: "TODO:\nBATTERY"
- note removed: "TODO:\nVBUS to OTF_FS_VBUS"
- moved on the sheet: C1, C10, C11, C12, C13, C14, C15, C16, C17, C18, C19, C2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

Commit message: Update footprint assignments
Parts:
- C1, C2, C3, C4, C5, C6: footprint (none) -> Capacitors_SMD:C_0402
- C22, C23, C24: footprint Capacitors_SMD:C_0402 -> (none)
- D1, D2: footprint LEDs:LED_0603 -> (none)
- J1: footprint (none) -> Connectors_Molex:USB_Micro-B_Molex_47346-0001
- J2: footprint (none) -> Pin_Headers:Pin_Header_Angled_1x02_Pitch2.54mm
- J3: footprint (none) -> Pin_Headers:Pin_Header_Angled_1x06_Pitch2.54mm
- J4: footprint (none) -> Pin_Headers:Pin_Header_Angled_1x03_Pitch2.54mm
- J5: footprint (none) -> Pin_Headers:Pin_Header_Angled_1x05_Pitch2.54mm
- R1, R2: footprint Resistors_SMD:R_0603 -> Resistors_SMD:R_0402
- R3, R4: footprint Resistors_SMD:R_0603 -> (none)
- U1: footprint (none) -> TO_SOT_Packages_SMD:TSOT-23-5_HandSoldering
- U2: footprint (none) -> Housings_DFN_QFN:QFN-32-1EP_5x5mm_Pitch0.5mm
- U4: footprint LQFP64 -> Housings_QFP:LQFP-64_10x10mm_Pitch0.5mm
- Y1: footprint Crystals:Crystal_SMD_0603-4pin_6.0x3.5mm -> (none)
- Y2: footprint Crystals:Crystal_AT310_d3.0mm_l10.0mm_Horizontal -> (none)

Commit message: CC1200 footprint
Parts:
- U2: footprint Housings_DFN_QFN:QFN-32-1EP_5x5mm_Pitch0.5mm -> CC1200:CC1200
Changed lines of the file:
@@
 EESchema Schematic File Version 2
-LIBS:RFM-rescue
 LIBS:power
 LIBS:device
@@
 F 0 "U2" H 8450 1075 60  0000 C CNN
 F 1 "CC1200" H 7775 2125 60  0000 C CNN
-F 2 "Housings_DFN_QFN:QFN-32-1EP_5x5mm_Pitch0.5mm" H 9125 2575 60  0001 C CNN
+F 2 "CC1200:CC1200" H 9125 2575 60  0001 C CNN
 F 3 "" H 9125 2575 60  0001 C CNN
 	1    7800 2125

Commit message: Balun footprint
Parts:
- C22, C23, C24: footprint (none) -> Capacitors_SMD:C_0603_HandSoldering
- D1, D2: footprint (none) -> LEDs:LED_0603
- R3, R4: footprint (none) -> Resistors_SMD:R_0603_HandSoldering
- U3: footprint (none) -> CC1200:BALF-112X-02D3
Changed lines of the file:
@@
 F 0 "U3" H 10275 2450 47  0000 C CNN
 F 1 "BALF-112X-02D3" H 9900 3000 47  0000 C CNN
-F 2 "" H 9925 2425 47  0001 C CNN
+F 2 "CC1200:BALF-112X-02D3" H 9925 2425 47  0001 C CNN
 F 3 "" H 9925 2425 47  0001 C CNN
 	1    9900 2800
@@
 F 0 "R3" V 3155 3075 50  0000 C CNN
 F 1 "200" V 3075 3075 50  0000 C CNN
-F 2 "" V 3005 3075 50  0001 C CNN
+F 2 "Resistors_SMD:R_0603_HandSoldering" V 3005 3075 50  0001 C CNN
 F 3 "" H 3075 3075 50  0000 C CNN
 	1    3075 3075
@@
 F 0 "C23" V 1025 4725 50  0000 L CNN
 F 1 "200" V 925 4725 50  0000 L CNN
-F 2 "" H 975 4900 50  0001 C CNN
+F 2 "Capacitors_SMD:C_0603_HandSoldering" H 975 4900 50  0001 C CNN
 F 3 "" H 975 4900 50  0000 C CNN
 	1    975  4900
@@
 F 0 "C24" V 1025 4925 50  0000 L CNN
 F 1 "200" V 925 4925 50  0000 L CNN
-F 2 "" H 975 5100 50  0001 C CNN
+F 2 "Capacitors_SMD:C_0603_HandSoldering" H 975 5100 50  0001 C CNN
 F 3 "" H 975 5100 50  0000 C CNN
 	1    975  5100
@@
 F 0 "D1" H 3375 3200 50  0000 L CNN
 F 1 "LED_PWR" H 3250 2975 50  0000 L CNN
-F 2 "" V 3425 3075 50  0001 C CNN
+F 2 "LEDs:LED_0603" V 3425 3075 50  0001 C CNN
 F 3 "" V 3425 3075 50  0000 C CNN
 	1    3425 3075
@@
 F 0 "C22" V 1075 3750 50  0000 L CNN
 F 1 "104/25V" V 1125 3400 50  0000 L CNN
-F 2 "" H 1025 3700 50  0001 C CNN
+F 2 "Capacitors_SMD:C_0603_HandSoldering" H 1025 3700 50  0001 C CNN
 F 3 "" H 1025 3700 50  0000 C CNN
 	1    1025 3700
@@
 F 0 "D2" H 6550 5525 50  0000 L CNN
 F 1 "LED_TEST" H 6425 5300 50  0000 L CNN
-F 2 "" V 6600 5400 50  0001 C CNN
+F 2 "LEDs:LED_0603" V 6600 5400 50  0001 C CNN
 F 3 "" V 6600 5400 50  0000 C CNN
 	1    6600 5400
@@
 F 0 "R4" V 6930 5400 50  0000 C CNN
 F 1 "200" V 6850 5400 50  0000 C CNN
-F 2 "" V 6780 5400 50  0001 C CNN
+F 2 "Resistors_SMD:R_0603_HandSoldering" V 6780 5400 50  0001 C CNN
 F 3 "" H 6850 5400 50  0000 C CNN
 	1    6850 5400

Commit message: Update footprints
Parts:
- removed SW1: SW_RESET, symbol SW_Push_Dual
- added SW1: SW_Push, Buttons_Switches_SMD:SW_SPST_PTS645, symbol SW_Push
- C22, C23, C24: footprint Capacitors_SMD:C_0603_HandSoldering -> Capacitors_SMD:C_0603
- L1: footprint (none) -> Inductors_SMD:L_0402
- P4: footprint (none) -> gsg-modules:SMA-EDGE
- R3, R4: footprint Resistors_SMD:R_0603_HandSoldering -> Resistors_SMD:R_0603
- U1: footprint TO_SOT_Packages_SMD:TSOT-23-5_HandSoldering -> TO_SOT_Packages_SMD:TSOT-23-5
- Y1: footprint (none) -> CC1200:NX3225SA-40M-EXS00A-CS03880
Connections:
- net GND: now also SW1.1
- net NRST: now also SW1.2
Changed lines of the file:
@@
 LIBS:switches
 LIBS:rfcom
+LIBS:gsg-symbols
 LIBS:RFM-cache
 EELAYER 25 0
@@
 F 0 "U1" H 4725 750 47  0000 C CNN
 F 1 "TPS79333" H 4450 975 47  0000 C CNN
-F 2 "TO_SOT_Packages_SMD:TSOT-23-5_HandSoldering" H 4425 1000 47  0001 C CNN
+F 2 "TO_SOT_Packages_SMD:TSOT-23-5" H 4425 1000 47  0001 C CNN
 F 3 "" H 4425 1000 47  0001 C CNN
 	1    4425 1000
@@
 F 0 "R3" V 3155 3075 50  0000 C CNN
 F 1 "200" V 3075 3075 50  0000 C CNN
-F 2 "Resistors_SMD:R_0603_HandSoldering" V 3005 3075 50  0001 C CNN
+F 2 "Resistors_SMD:R_0603" V 3005 3075 50  0001 C CNN
 F 3 "" H 3075 3075 50  0000 C CNN
 	1    3075 3075
@@
 F 0 "C23" V 1025 4725 50  0000 L CNN
 F 1 "200" V 925 4725 50  0000 L CNN
-F 2 "Capacitors_SMD:C_0603_HandSoldering" H 975 4900 50  0001 C CNN
+F 2 "Capacitors_SMD:C_0603" H 975 4900 50  0001 C CNN
 F 3 "" H 975 4900 50  0000 C CNN
 	1    975  4900
@@
 F 0 "C24" V 1025 4925 50  0000 L CNN
 F 1 "200" V 925 4925 50  0000 L CNN
-F 2 "Capacitors_SMD:C_0603_HandSoldering" H 975 5100 50  0001 C CNN
+F 2 "Capacitors_SMD:C_0603" H 975 5100 50  0001 C CNN
 F 3 "" H 975 5100 50  0000 C CNN
 	1    975  5100
@@
 F 0 "Y1" V 9225 2000 50  0000 L CNN
 F 1 "40MHz" V 8975 1775 50  0000 L CNN
-F 2 "" H 9175 1900 50  0001 C CNN
+F 2 "CC1200:NX3225SA-40M-EXS00A-CS03880" H 9175 1900 50  0001 C CNN
 F 3 "" H 9175 1900 50  0000 C CNN
 	1    9175 1900
@@
 F 0 "L1" H 9155 3615 50  0000 L CNN
 F 1 "56nH" H 9155 3535 50  0000 L CNN
-F 2 "" H 9125 3575 50  0001 C CNN
+F 2 "Inductors_SMD:L_0402" H 9125 3575 50  0001 C CNN
 F 3 "" H 9125 3575 50  0000 C CNN
 	1    9125 3575
@@
 $EndComp
 $Comp
-L SW_Push_Dual SW1
-U 1 1 58C2D4C2
-P 1025 3350
-F 0 "SW1" H 1075 3450 50  0000 L CNN
-F 1 "SW_RESET" H 1025 3550 50  0000 C CNN
-F 2 "" H 1025 3550 50  0001 C CNN
-F 3 "" H 1025 3550 50  0000 C CNN
-	1    1025 3350
-	1    0    0    -1
-$EndComp
-$Comp
 L GND #PWR041
 U 1 1 58C2E4FB
@@
 F 0 "C22" V 1075 3750 50  0000 L CNN
 F 1 "104/25V" V 1125 3400 50  0000 L CNN
-F 2 "Capacitors_SMD:C_0603_HandSoldering" H 1025 3700 50  0001 C CNN
+F 2 "Capacitors_SMD:C_0603" H 1025 3700 50  0001 C CNN
 F 3 "" H 1025 3700 50  0000 C CNN
 	1    1025 3700
@@
 F 0 "R4" V 6930 5400 50  0000 C CNN
 F 1 "200" V 6850 5400 50  0000 C CNN
-F 2 "Resistors_SMD:R_0603_HandSoldering" V 6780 5400 50  0001 C CNN
+F 2 "Resistors_SMD:R_0603" V 6780 5400 50  0001 C CNN
 F 3 "" H 6850 5400 50  0000 C CNN
 	1    6850 5400
@@
 Text GLabel 6500 6900 2    47   Input ~ 0
 SPI_MOSI
+Text GLabel 2975 1275 0    47   Input ~ 0
+SPI_NSS
+Text GLabel 2975 1375 0    47   Input ~ 0
+SPI_SCK
+Text GLabel 2975 1475 0    47   Input ~ 0
+SPI_MISO
+Text GLabel 2975 1575 0    47   Input ~ 0
+SPI_MOSI
+$Comp
+L CONN_01X05 J5
+U 1 1 58C52067
+P 3175 1475
+F 0 "J5" H 3175 1775 50  0000 C CNN
+F 1 "CONN_SPI" H 3050 1175 50  0000 C CNN
+F 2 "Pin_Headers:Pin_Header_Angled_1x05_Pitch2.54mm" H 3175 1475 50  0001 C CNN
+F 3 "" H 3175 1475 50  0001 C CNN
+	1    3175 1475
+	1    0    0    -1
+$EndComp
+$Comp
+L GND #PWR069
+U 1 1 58C52138
+P 2975 1675
+F 0 "#PWR069" H 2975 1425 50  0001 C CNN
+F 1 "GND" V 2975 1475 50  0000 C CNN
+F 2 "" H 2975 1675 50  0000 C CNN
+F 3 "" H 2975 1675 50  0000 C CNN
+	1    2975 1675
+	0    1    1    0
+$EndComp
+$Comp
+L CONN_01X03 J4
+U 1 1 58C525A3
+P 3175 825
+F 0 "J4" H 3175 1025 50  0000 C CNN
+F 1 "CONN_USART" H 3000 625 50  0000 C CNN
+F 2 "Pin_Headers:Pin_Header_Angled_1x03_Pitch2.54mm" H 3175 825 50  0001 C CNN
+F 3 "" H 3175 825 50  0001 C CNN
+	1    3175 825
+	1    0    0    -1
+$EndComp
+$Comp
+L GND #PWR070
+U 1 1 58C5290D
+P 2975 925
+F 0 "#PWR070" H 2975 675 50  0001 C CNN
+F 1 "GND" V 2975 725 50  0000 C CNN
+F 2 "" H 2975 925 50  0000 C CNN
+F 3 "" H 2975 925 50  0000 C CNN
+	1    2975 925
+	0    1    1    0
+$EndComp
+$Comp
+L CONN_01X02 J2
+U 1 1 58C52D4E
+P 2300 775
+F 0 "J2" H 2300 925 50  0000 C CNN
+F 1 "CONN_PWR" H 2150 625 50  0000 C CNN
+F 2 "Pin_Headers:Pin_Header_Angled_1x02_Pitch2.54mm" H 2300 775 50  0001 C CNN
+F 3 "" H 2300 775 50  0001 C CNN
+	1    2300 775
+	1    0    0    -1
+$EndComp
+$Comp
+L CONN_01X06 J3
+U 1 1 58C52EE6
+P 2300 1425
+F 0 "J3" H 2300 1775 50  0000 C CNN
+F 1 "CONN_DEBUG" H 2125 1075 50  0000 C CNN
+F 2 "Pin_Headers:Pin_Header_Angled_1x06_Pitch2.54mm" H 2300 1425 50  0001 C CNN
+F 3 "" H 2300 1425 50  0001 C CNN
+	1    2300 1425
+	1    0    0    -1
+$EndComp
+$Comp
+L BNC P4
+U 1 1 58C37BB0
+P 11000 2850
+F 0 "P4" H 11010 2970 50  0000 C CNN
+F 1 "SMA" H 11100 2750 50  0000 C CNN
+F 2 "gsg-modules:SMA-EDGE" H 11000 2850 50  0001 C CNN
+F 3 "" H 11000 2850 50  0000 C CNN
+	1    11000 2850
+	1    0    0    -1
+$EndComp
+Text Notes 4325 2975 0    60   ~ 0
+TODO: decoupling
+$Comp
+L SW_Push SW1
+U 1 1 58CBA9FF
+P 1025 3525
+F 0 "SW1" H 1075 3625 50  0000 L CNN
+F 1 "SW_Push" H 1025 3465 50  0000 C CNN
+F 2 "Buttons_Switches_SMD:SW_SPST_PTS645" H 1025 3725 50  0001 C CNN
+F 3 "" H 1025 3725 50  0001 C CNN
+	1    1025 3525
+	1    0    0    -1
+$EndComp
 Wire Wire Line
 	1150 1225 1150 1425
@@
 	1350 4100 1525 4100
 Wire Wire Line
-	1225 3350 1225 3700
-Connection ~ 825  3550
-Wire Wire Line
 	750  3700 925  3700
 Wire Wire Line
 	1125 3700 1525 3700
-Connection ~ 1225 3550
 Connection ~ 1225 3700
-Wire Wire Line
-	825  3350 825  3700
 Connection ~ 825  3700
 Wire Wire Line
@@
 Wire Wire Line
 	6325 6900 6500 6900
-Text GLabel 2975 1275 0    47   Input ~ 0
-SPI_NSS
-Text GLabel 2975 1375 0    47   Input ~ 0
-SPI_SCK
-Text GLabel 2975 1475 0    47   Input ~ 0
-SPI_MISO
-Text GLabel 2975 1575 0    47   Input ~ 0
-SPI_MOSI
-$Comp
-L CONN_01X05 J5
-U 1 1 58C52067
-P 3175 1475
-F 0 "J5" H 3175 1775 50  0000 C CNN
-F 1 "CONN_SPI" H 3050 1175 50  0000 C CNN
-F 2 "Pin_Headers:Pin_Header_Angled_1x05_Pitch2.54mm" H 3175 1475 50  0001 C CNN
-F 3 "" H 3175 1475 50  0001 C CNN
-	1    3175 1475
-	1    0    0    -1
-$EndComp
-$Comp
-L GND #PWR069
-U 1 1 58C52138
-P 2975 1675
-F 0 "#PWR069" H 2975 1425 50  0001 C CNN
-F 1 "GND" V 2975 1475 50  0000 C CNN
-F 2 "" H 2975 1675 50  0000 C CNN
-F 3 "" H 2975 1675 50  0000 C CNN
-	1    2975 1675
-	0    1    1    0
-$EndComp
-$Comp
-L CONN_01X03 J4
-U 1 1 58C525A3
-P 3175 825
-F 0 "J4" H 3175 1025 50  0000 C CNN
-F 1 "CONN_USART" H 3000 625 50  0000 C CNN
-F 2 "Pin_Headers:Pin_Header_Angled_1x03_Pitch2.54mm" H 3175 825 50  0001 C CNN
-F 3 "" H 3175 825 50  0001 C CNN
-	1    3175 825
-	1    0    0    -1
-$EndComp
-$Comp
-L GND #PWR070
-U 1 1 58C5290D
-P 2975 925
-F 0 "#PWR070" H 2975 675 50  0001 C CNN
-F 1 "GND" V 2975 725 50  0000 C CNN
-F 2 "" H 2975 925 50  0000 C CNN
-F 3 "" H 2975 925 50  0000 C CNN
-	1    2975 925
-	0    1    1    0
-$EndComp
-$Comp
-L CONN_01X02 J2
-U 1 1 58C52D4E
-P 2300 775
-F 0 "J2" H 2300 925 50  0000 C CNN
-F 1 "CONN_PWR" H 2150 625 50  0000 C CNN
-F 2 "Pin_Headers:Pin_Header_Angled_1x02_Pitch2.54mm" H 2300 775 50  0001 C CNN
-F 3 "" H 2300 775 50  0001 C CNN
-	1    2300 775
-	1    0    0    -1
-$EndComp
-$Comp
-L CONN_01X06 J3
-U 1 1 58C52EE6
-P 2300 1425
-F 0 "J3" H 2300 1775 50  0000 C CNN
-F 1 "CONN_DEBUG" H 2125 1075 50  0000 C CNN
-F 2 "Pin_Headers:Pin_Header_Angled_1x06_Pitch2.54mm" H 2300 1425 50  0001 C CNN
-F 3 "" H 2300 1425 50  0001 C CNN
-	1    2300 1425
-	1    0    0    -1
-$EndComp
-$Comp
-L BNC P4
-U 1 1 58C37BB0
-P 11000 2850
-F 0 "P4" H 11010 2970 50  0000 C CNN
-F 1 "SMA" H 11100 2750 50  0000 C CNN
-F 2 "" H 11000 2850 50  0001 C CNN
-F 3 "" H 11000 2850 50  0000 C CNN
-	1    11000 2850
-	1    0    0    -1
-$EndComp
-Text Notes 4325 2975 0    60   ~ 0
-TODO: decoupling
+Wire Wire Line
+	1225 3700 1225 3525
+Wire Wire Line
+	825  3700 825  3525
 $EndSCHEMATC
