File: cc.kicad_pcb (KiCad board)
At the start: 2 copper layers, 44 parts, among them J1 USB_OTG, J2 CONN_PWR, J3 CONN_DEBUG, J4 CONN_USART, J5 CONN_SPI, P4 SMA, SW1 SW_Push, U1 TPS79333, U2 CC1200, U3 BALF-112X-02D3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

Commit message: Rename
Parts:
- removed P4: SMA, gsg-modules:SMA-EDGE
- added P1: SMA, gsg-modules:SMA-EDGE, F.Cu at (182.9, 117.6)
- moved C10 46.2 mm to (229.8, 100.9)
- moved C11 46.2 mm to (212.5, 119.7)
- moved C14 46.2 mm to (208.4, 119.7)
- moved C16 46.2 mm to (226.2, 95.4)
- moved C22 46.2 mm to (212.2, 105.7)
- moved C5 46.2 mm to (216.5, 119.7)
- moved C9 46.2 mm to (216.6, 115.1)
- moved D1 46.2 mm to (225.6, 90.7)
- moved J5 46.2 mm to (172.0, 106.4)
- moved R1 46.2 mm to (188.3, 116.5)
- moved R2 46.2 mm to (235.1, 86.1)
- moved U1 46.2 mm to (193.9, 115.4)
- moved U2 46.2 mm to (205.4, 104.0)
- moved U3 46.2 mm to (202.8, 86.9)
- moved Y1 46.2 mm to (200.5, 115.4)
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Other:
- rule pad_to_mask_clearance: 0.2 -> 0
