File: cc.sch (KiCad schematic (older format))
At the start: 44 parts, among them J1 USB_OTG, J2 CONN_PWR, J3 CONN_DEBUG, J4 CONN_USART, J5 CONN_SPI, P4 SMA, SW1 SW_Push, U1 TPS79333, U2 CC1200, U3 BALF-112X-02D3, U4 STM32F103R8Tx, Y1 40MHz, Y2 8MHz(16pF)

Commit message: Rename
Parts:
- removed P4: SMA, gsg-modules:SMA-EDGE, symbol BNC
- added P1: SMA, gsg-modules:SMA-EDGE, symbol SMA
- Y2: footprint (none) -> Crystals:Crystal_SMD_HC49-SD
Changed lines of the file:
@@
 LIBS:contrib
 LIBS:valves
-LIBS:RFM
 LIBS:stm32
 LIBS:switches
-LIBS:rfcom
 LIBS:gsg-symbols
-LIBS:RFM-cache
+LIBS:cclib
 EELAYER 25 0
 EELAYER END
@@
 F 0 "Y2" V 1225 4875 50  0000 C CNN
 F 1 "8MHz(16pF)" V 1400 4875 50  0000 C CNN
-F 2 "" H 1225 5000 50  0001 C CNN
+F 2 "Crystals:Crystal_SMD_HC49-SD" H 1225 5000 50  0001 C CNN
 F 3 "" H 1225 5000 50  0000 C CNN
 	1    1225 5000
@@
 	1    0    0    -1
 $EndComp
-$Comp
-L BNC P4
-U 1 1 58C37BB0
-P 11000 2850
-F 0 "P4" H 11010 2970 50  0000 C CNN
-F 1 "SMA" H 11100 2750 50  0000 C CNN
-F 2 "gsg-modules:SMA-EDGE" H 11000 2850 50  0001 C CNN
-F 3 "" H 11000 2850 50  0000 C CNN
-	1    11000 2850
-	1    0    0    -1
-$EndComp
 Text Notes 4325 2975 0    60   ~ 0
 TODO: decoupling
@@
 Wire Wire Line
 	825  3700 825  3525
+$Comp
+L SMA P1
+U 1 1 58CBB947
+P 11000 2850
+F 0 "P1" H 11010 2970 50  0000 C CNN
+F 1 "SMA" H 11100 2750 50  0000 C CNN
+F 2 "gsg-modules:SMA-EDGE" H 11000 2850 50  0001 C CNN
+F 3 "" H 11000 2850 50  0000 C CNN
+	1    11000 2850
+	1    0    0    -1
+$EndComp
 $EndSCHEMATC

Commit message: Use STM32L475RC
Parts:
- removed U4: STM32F103R8Tx, Housings_QFP:LQFP-64_10x10mm_Pitch0.5mm, symbol STM32F103R8Tx
- added R3: 10k, Resistors_SMD:R_0603, symbol R_Small
- added SW2: SW_Push, Buttons_Switches_SMD:SW_SPST_PTS645, symbol SW_Push
- added U4: STM32L475RC, Housings_QFP:LQFP-64_10x10mm_Pitch0.5mm, symbol STM32L475RC
- C4: renamed from C22; value 104/25V -> 0.1uF/25V
- C5: renamed from C23; value 200 -> 20pF
- C6: renamed from C24; value 200 -> 20pF
- renumbered C12 to C11, C10 to C121, C9 to C131, C8 to C151, C17 to C173, C16 to C17A1, C3 to C2, C19 to C211, C5 to C221, C15 to C231, C7 to C251, C20 to C261, C4 to C271, C6 to C281, C21 to C291, C2 to C3, C13 to C301, C14 to C311, C11 to C51, C18 to C61, L1 to L171, R3 to R1, R2 to R141, R1 to R171, R4 to R2
Connections:
- net CC_GPIO0: now also U4.41 (PA8)
- net CC_GPIO2: now also U4.14 (PA0)
- net CC_GPIO3: now also U4.15 (PA1)
- net CC_MISO: now also U4.22 (PA6)
- net CC_MOSI: now also U4.23 (PA7)
- net CC_NSS: now also U4.20 (PA4)
- net CC_RESET_N: now also U4.42 (PA9)
- net CC_SCLK: now also U4.21 (PA5)
- net GND: now also C4.1, SW1.2, R3.2, U4.18 (VSS), U4.31 (VSS), U4.47 (VSS), U4.63 (VSS); no longer C4.2, SW1.1
- net NRST: now also C4.2, SW1.1, U4.7 (NRST); no longer C4.1, SW1.2
- net SPI_MISO: now also U4.35 (PB14)
- net SPI_MOSI: now also U4.36 (PB15)
- net SPI_NSS: now also U4.33 (PB12)
- net SPI_SCK: now also U4.34 (PB13)
- net SWDIO: now also U4.46 (PA13/SWDIO)
- net SWO: now also U4.55 (PB3/SWO)
- net USART_RX: now also U4.17 (PA3)
- net USART_TX: now also U4.16 (PA2)
- net USB_DM: now also U4.44 (PA11)
- net USB_DP: now also U4.45 (PA12)
- net USB_ID: now also U4.43 (PA10)
- net VDD: now also SW2.1, U4.1 (VBAT), U4.19 (VDD), U4.32 (VDD), U4.48 (VDDUSB), U4.64 (VDD)
- net VDDA: now also U4.13 (VDDA)
- net VSSA: now also U4.12 (VSSA)
- net at D2.2 (A): now also U4.59 (PB7)
- net at C5.1, Y2.2: now also U4.5 (PH0/OSC_IN)
- net at C6.1, Y2.1: now also U4.6 (PH1/OSC_OUT)
- net SWDCLK renamed SWCLK
- net SWCLK: now also U4.49 (PA14/SWCLK)
- new net: R3.1, SW2.2, U4.60 (BOOT0)
Other:
- note added: "TODO: Front end, GPS, STM32F207VC, DCMI, \nuBLOX NEO-6Q/MAX-6Q\n\n"
- note removed: "TODO: Front end, GPS"
- moved on the sheet: C11, C121, C131, C151, C173, C17A1, C211, C221, C231, C251, C261, C271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

Commit message: Footprint spreadout
Connections:
- net SPI_MISO: now also J5.2 (P2); no longer J5.3 (P3)
- net SPI_MOSI: now also J5.1 (P1); no longer J5.4 (P4)
- net SPI_NSS: now also J5.4 (P4); no longer J5.1 (P1)
- net SPI_SCK: now also J5.3 (P3); no longer J5.2 (P2)
- net USART_RX: now also J4.1 (P1); no longer J4.2 (P2)
- net USART_TX: now also J4.2 (P2); no longer J4.1 (P1)
Changed lines of the file:
@@
 	0    -1   -1   0
 $EndComp
+Text GLabel 2975 825  0    47   Input ~ 0
+USART_TX
 Text GLabel 2975 725  0    47   Input ~ 0
-USART_TX
-Text GLabel 2975 825  0    47   Input ~ 0
 USART_RX
 Text GLabel 1600 3725 0    47   Input ~ 0
@@
 SPI_MOSI
 Text GLabel 2975 1275 0    47   Input ~ 0
+SPI_MOSI
+Text GLabel 2975 1375 0    47   Input ~ 0
+SPI_MISO
+Text GLabel 2975 1475 0    47   Input ~ 0
+SPI_SCK
+Text GLabel 2975 1575 0    47   Input ~ 0
 SPI_NSS
-Text GLabel 2975 1375 0    47   Input ~ 0
-SPI_SCK
-Text GLabel 2975 1475 0    47   Input ~ 0
-SPI_MISO
-Text GLabel 2975 1575 0    47   Input ~ 0
-SPI_MOSI
 $Comp
 L CONN_01X05 J5

Commit message: PCB layout WIP
Connections:
- net CC_GPIO0: now also U4.14 (PA0); no longer U4.41 (PA8)
- net CC_GPIO2: now also U4.28 (PB2); no longer U4.14 (PA0)
- net CC_GPIO3: now also U4.29 (PB10); no longer U4.15 (PA1)
- net CC_RESET_N: now also U4.30 (PB11); no longer U4.42 (PA9)
- net USART_RX: now also U4.59 (PB7); no longer U4.17 (PA3)
- net USART_TX: now also U4.58 (PB6); no longer U4.16 (PA2)
- net at D2.2 (A): now also U4.54 (PD2); no longer U4.59 (PB7)
Other:
- moved on the sheet: D2, R2
Changed lines of the file:
@@
 Text GLabel 1600 4525 0    47   Input ~ 0
 SWCLK
-Text GLabel 1600 3425 0    47   Input ~ 0
+Text GLabel 1600 5550 0    47   Input ~ 0
 USART_RX
-Text GLabel 1600 3325 0    47   Input ~ 0
+Text GLabel 1600 5450 0    47   Input ~ 0
 USART_TX
 $Comp
@@
 Text GLabel 1600 3525 0    47   Input ~ 0
 CC_NSS
-Text GLabel 1600 4025 0    47   Input ~ 0
+Text GLabel 1600 5950 0    47   Input ~ 0
 CC_RESET_N
-Text GLabel 1600 3925 0    47   Input ~ 0
+Text GLabel 1600 3125 0    47   Input ~ 0
 CC_GPIO0
-Text GLabel 1600 3125 0    47   Input ~ 0
+Text GLabel 1600 5050 0    47   Input ~ 0
 CC_GPIO2
 $Comp
@@
 L LED_Small_ALT D2
 U 1 1 58C31362
-P 1500 5550
-F 0 "D2" H 1450 5675 50  0000 L CNN
-F 1 "LED_TEST" H 1325 5450 50  0000 L CNN
-F 2 "LEDs:LED_0603" V 1500 5550 50  0001 C CNN
-F 3 "" V 1500 5550 50  0000 C CNN
-	1    1500 5550
-	1    0    0    -1
+P 3725 6275
+F 0 "D2" H 3675 6400 50  0000 L CNN
+F 1 "LED_TEST" H 3550 6175 50  0000 L CNN
+F 2 "LEDs:LED_0603" V 3725 6275 50  0001 C CNN
+F 3 "" V 3725 6275 50  0000 C CNN
+	1    3725 6275
+	-1   0    0    1
 $EndComp
 $Comp
 L R R2
 U 1 1 58C31AFC
-P 1250 5550
-F 0 "R2" V 1330 5550 50  0000 C CNN
-F 1 "200" V 1250 5550 50  0000 C CNN
-F 2 "Resistors_SMD:R_0603" V 1180 5550 50  0001 C CNN
-F 3 "" H 1250 5550 50  0000 C CNN
-	1    1250 5550
-	0    -1   -1   0
+P 3975 6275
+F 0 "R2" V 4055 6275 50  0000 C CNN
+F 1 "200" V 3975 6275 50  0000 C CNN
+F 2 "Resistors_SMD:R_0603" V 3905 6275 50  0001 C CNN
+F 3 "" H 3975 6275 50  0000 C CNN
+	1    3975 6275
+	0    1    1    0
 $EndComp
 $Comp
 L GND #PWR039
 U 1 1 58C31BFA
-P 975 5550
-F 0 "#PWR039" H 975 5300 50  0001 C CNN
-F 1 "GND" H 975 5400 50  0000 C CNN
-F 2 "" H 975 5550 50  0000 C CNN
-F 3 "" H 975 5550 50  0000 C CNN
-	1    975  5550
+P 4250 6275
+F 0 "#PWR039" H 4250 6025 50  0001 C CNN
+F 1 "GND" H 4250 6125 50  0000 C CNN
+F 2 "" H 4250 6275 50  0000 C CNN
+F 3 "" H 4250 6275 50  0000 C CNN
+	1    4250 6275
 	1    0    0    -1
 $EndComp
@@
 	1    0    0    -1
 $EndComp
-Text GLabel 1600 3225 0    47   Input ~ 0
+Text GLabel 1600 5850 0    47   Input ~ 0
 CC_GPIO3
 Text Notes 4075 725  0    60   ~ 0
@@
 NoConn ~ 1775 4850
 NoConn ~ 1775 4950
-NoConn ~ 1775 5050
 NoConn ~ 1775 5250
 NoConn ~ 1775 5350
-NoConn ~ 1775 5450
 NoConn ~ 1775 5650
 NoConn ~ 1775 5750
-NoConn ~ 1775 5850
-NoConn ~ 1775 5950
 NoConn ~ 4525 4450
 NoConn ~ 4525 4550
@@
 NoConn ~ 4525 5850
 NoConn ~ 4525 5950
-NoConn ~ 3450 6275
 $Comp
 L SW_Push SW2
@@
 Connection ~ 5025 4025
 Wire Wire Line
-	1775 5550 1600 5550
-Wire Wire Line
-	1100 5550 975  5550
+	3450 6275 3625 6275
+Wire Wire Line
+	4125 6275 4250 6275
 Wire Wire Line
 	10400 4275 10700 4275
@@
 Connection ~ 700  925
 Wire Wire Line
+	1600 5550 1775 5550
+Wire Wire Line
 	1600 3125 1775 3125
 Wire Wire Line
-	1600 3425 1775 3425
-Wire Wire Line
-	1600 4025 1775 4025
-Wire Wire Line
-	1600 3925 1775 3925
-Wire Wire Line
 	1775 3825 1600 3825
 Wire Wire Line
@@
 	1600 4425 1775 4425
 Wire Wire Line
-	1775 3225 1600 3225
-Wire Wire Line
-	1775 3325 1600 3325
+	1775 5450 1600 5450
 Wire Wire Line
 	1600 4125 1775 4125
@@
 Wire Wire Line
 	3100 6350 3150 6350
+Wire Wire Line
+	1600 5050 1775 5050
+Wire Wire Line
+	1600 5850 1775 5850
+Wire Wire Line
+	1600 5950 1775 5950
+NoConn ~ 1775 3925
+NoConn ~ 1775 3225
+NoConn ~ 1775 4025
+NoConn ~ 1775 3325
+NoConn ~ 1775 3425
 $EndSCHEMATC

Commit message: Component layout etc.
Parts:
- removed J5: CONN_SPI, Pin_Headers:Pin_Header_Angled_1x05_Pitch2.54mm, symbol CONN_01X05
- J2: footprint Pin_Headers:Pin_Header_Angled_1x02_Pitch2.54mm -> Pin_Headers:Pin_Header_Straight_1x02_Pitch1.27mm
- J3: footprint Pin_Headers:Pin_Header_Angled_1x06_Pitch2.54mm -> Pin_Headers:Pin_Header_Straight_1x06_Pitch1.27mm
- J4: footprint Pin_Headers:Pin_Header_Angled_1x03_Pitch2.54mm -> Pin_Headers:Pin_Header_Straight_1x03_Pitch1.27mm
Changed lines of the file:
@@
 Text GLabel 4700 3625 2    47   Input ~ 0
 SPI_MOSI
-Text GLabel 2975 1275 0    47   Input ~ 0
-SPI_MOSI
-Text GLabel 2975 1375 0    47   Input ~ 0
-SPI_MISO
-Text GLabel 2975 1475 0    47   Input ~ 0
-SPI_SCK
-Text GLabel 2975 1575 0    47   Input ~ 0
-SPI_NSS
-$Comp
-L CONN_01X05 J5
-U 1 1 58C52067
-P 3175 1475
-F 0 "J5" H 3175 1775 50  0000 C CNN
-F 1 "CONN_SPI" H 3050 1175 50  0000 C CNN
-F 2 "Pin_Headers:Pin_Header_Angled_1x05_Pitch2.54mm" H 3175 1475 50  0001 C CNN
-F 3 "" H 3175 1475 50  0001 C CNN
-	1    3175 1475
-	1    0    0    -1
-$EndComp
-$Comp
-L GND #PWR065
-U 1 1 58C52138
-P 2975 1675
-F 0 "#PWR065" H 2975 1425 50  0001 C CNN
-F 1 "GND" V 2975 1475 50  0000 C CNN
-F 2 "" H 2975 1675 50  0000 C CNN
-F 3 "" H 2975 1675 50  0000 C CNN
-	1    2975 1675
-	0    1    1    0
-$EndComp
 $Comp
 L CONN_01X03 J4
@@
 F 0 "J4" H 3175 1025 50  0000 C CNN
 F 1 "CONN_USART" H 3000 625 50  0000 C CNN
-F 2 "Pin_Headers:Pin_Header_Angled_1x03_Pitch2.54mm" H 3175 825 50  0001 C CNN
+F 2 "Pin_Headers:Pin_Header_Straight_1x03_Pitch1.27mm" H 3175 825 50  0001 C CNN
 F 3 "" H 3175 825 50  0001 C CNN
 	1    3175 825
@@
 $EndComp
 $Comp
-L GND #PWR066
+L GND #PWR065
 U 1 1 58C5290D
 P 2975 925
-F 0 "#PWR066" H 2975 675 50  0001 C CNN
+F 0 "#PWR065" H 2975 675 50  0001 C CNN
 F 1 "GND" V 2975 725 50  0000 C CNN
 F 2 "" H 2975 925 50  0000 C CNN
@@
 F 0 "J2" H 2300 925 50  0000 C CNN
 F 1 "CONN_PWR" H 2150 625 50  0000 C CNN
-F 2 "Pin_Headers:Pin_Header_Angled_1x02_Pitch2.54mm" H 2300 775 50  0001 C CNN
+F 2 "Pin_Headers:Pin_Header_Straight_1x02_Pitch1.27mm" H 2300 775 50  0001 C CNN
 F 3 "" H 2300 775 50  0001 C CNN
 	1    2300 775
@@
 F 0 "J3" H 2300 1775 50  0000 C CNN
 F 1 "CONN_DEBUG" H 2125 1075 50  0000 C CNN
-F 2 "Pin_Headers:Pin_Header_Angled_1x06_Pitch2.54mm" H 2300 1425 50  0001 C CNN
+F 2 "Pin_Headers:Pin_Header_Straight_1x06_Pitch1.27mm" H 2300 1425 50  0001 C CNN
 F 3 "" H 2300 1425 50  0001 C CNN
 	1    2300 1425
@@
 $EndComp
 $Comp
-L VDD #PWR067
+L VDD #PWR066
 U 1 1 58CD6E6D
 P 2375 6375
-F 0 "#PWR067" H 2375 6225 50  0001 C CNN
+F 0 "#PWR066" H 2375 6225 50  0001 C CNN
 F 1 "VDD" H 2375 6525 50  0000 C CNN
 F 2 "" H 2375 6375 50  0000 C CNN
@@
 $EndComp
 $Comp
-L VDD #PWR068
+L VDD #PWR067
 U 1 1 58CD6EFA
 P 2925 2675
-F 0 "#PWR068" H 2925 2525 50  0001 C CNN
+F 0 "#PWR067" H 2925 2525 50  0001 C CNN
 F 1 "VDD" H 2925 2825 50  0000 C CNN
 F 2 "" H 2925 2675 50  0000 C CNN
@@
 $EndComp
 $Comp
-L GND #PWR069
+L GND #PWR068
 U 1 1 58CD7406
 P 2750 2675
-F 0 "#PWR069" H 2750 2425 50  0001 C CNN
+F 0 "#PWR068" H 2750 2425 50  0001 C CNN
 F 1 "GND" H 2750 2525 50  0000 C CNN
 F 2 "" H 2750 2675 50  0001 C CNN
@@
 $EndComp
 $Comp
-L GND #PWR070
+L GND #PWR069
 U 1 1 58CD80A9
 P 3150 2675
-F 0 "#PWR070" H 3150 2425 50  0001 C CNN
+F 0 "#PWR069" H 3150 2425 50  0001 C CNN
 F 1 "GND" H 3150 2525 50  0000 C CNN
 F 2 "" H 3150 2675 50  0001 C CNN
@@
 $EndComp
 $Comp
-L GND #PWR071
+L GND #PWR070
 U 1 1 58CD8138
 P 3950 2675
-F 0 "#PWR071" H 3950 2425 50  0001 C CNN
+F 0 "#PWR070" H 3950 2425 50  0001 C CNN
 F 1 "GND" H 3950 2525 50  0000 C CNN
 F 2 "" H 3950 2675 50  0001 C CNN
@@
 $EndComp
 $Comp
-L GND #PWR072
+L GND #PWR071
 U 1 1 58CD81C7
 P 3550 2675
-F 0 "#PWR072" H 3550 2425 50  0001 C CNN
+F 0 "#PWR071" H 3550 2425 50  0001 C CNN
 F 1 "GND" H 3550 2525 50  0000 C CNN
 F 2 "" H 3550 2675 50  0001 C CNN
@@
 $EndComp
 $Comp
-L VDD #PWR073
+L VDD #PWR072
 U 1 1 58CD8256
 P 3725 2675
-F 0 "#PWR073" H 3725 2525 50  0001 C CNN
+F 0 "#PWR072" H 3725 2525 50  0001 C CNN
 F 1 "VDD" H 3725 2825 50  0000 C CNN
 F 2 "" H 3725 2675 50  0000 C CNN
@@
 $EndComp
 $Comp
-L VSSA #PWR074
+L VSSA #PWR073
 U 1 1 58CD8A59
 P 2325 2675
-F 0 "#PWR074" H 2325 2525 50  0001 C CNN
+F 0 "#PWR073" H 2325 2525 50  0001 C CNN
 F 1 "VSSA" H 2325 2825 50  0000 C CNN
 F 2 "" H 2325 2675 50  0001 C CNN
@@
 $EndComp
 $Comp
-L VDD #PWR075
+L VDD #PWR074
 U 1 1 58CD9729
 P 6600 700
-F 0 "#PWR075" H 6600 550 50  0001 C CNN
+F 0 "#PWR074" H 6600 550 50  0001 C CNN
 F 1 "VDD" H 6600 850 50  0000 C CNN
 F 2 "" H 6600 700 50  0000 C CNN
@@
 $EndComp
 $Comp
-L VDD #PWR076
+L VDD #PWR075
 U 1 1 58CCEB62
 P 4150 2675
-F 0 "#PWR076" H 4150 2525 50  0001 C CNN
+F 0 "#PWR075" H 4150 2525 50  0001 C CNN
 F 1 "VDD" H 4150 2825 50  0000 C CNN
 F 2 "" H 4150 2675 50  0000 C CNN
@@
 $EndComp
 $Comp
-L GND #PWR077
+L GND #PWR076
 U 1 1 58CD7242
 P 2325 7275
-F 0 "#PWR077" H 2325 7025 50  0001 C CNN
+F 0 "#PWR076" H 2325 7025 50  0001 C CNN
 F 1 "GND" H 2325 7125 50  0000 C CNN
 F 2 "" H 2325 7275 50  0000 C CNN
@@
 $EndComp
 $Comp
-L VDD #PWR078
+L VDD #PWR077
 U 1 1 58CD7576
 P 1850 6825
-F 0 "#PWR078" H 1850 6675 50  0001 C CNN
+F 0 "#PWR077" H 1850 6675 50  0001 C CNN
 F 1 "VDD" H 1850 6975 50  0000 C CNN
 F 2 "" H 1850 6825 50  0000 C CNN

Commit message: Pre v0.1.0
Other:
- note added: "TODO: Front end, Camera,\nuBLOX NEO-6Q/MAX-6Q\n\n"
- note removed: "TODO: Front end, GPS, STM32F207VC, DCMI, \nuBLOX NEO-6Q/MAX-6Q\n\n"
Changed lines of the file:
@@
 Linear regulator
 Text Notes 9125 6525 0    60   ~ 0
-TODO: Front end, GPS, STM32F207VC, DCMI, \nuBLOX NEO-6Q/MAX-6Q\n\n
+TODO: Front end, Camera,\nuBLOX NEO-6Q/MAX-6Q\n\n
 Text Notes 3925 1850 0    60   ~ 0
 Consider using LP38798
